File: Motor Driver/1-Axis Reaction Wheel/Avionics-RWboard-main/Avionics-RWboard.kicad_pcb (KiCad board)
At the start: 4 copper layers, 90.2 x 95.9 mm, 135 parts, among them J1 Input Power, J2 522711069, M1 304D-262503, Q1 NX3008NBKS, Q10 MBT2222ADW1T1, Q11 NX3008NBKS, Q12 MBT2222ADW1T1, Q2 MBT2222ADW1T1, Q3 NX3008NBKS, Q4 MBT2222ADW1T1, Q5 IRLML2803, Q6 SiRA99DP, Q9 NX3008NBKS, U1 MCF8315C1VQRGFRQ1, U2 TPS259621DDA, U3 NCP730BMT330TBG, U4 ADM1176-1ARMZ-R7

Commit message: Review changes
Parts:
- moved REF** 66.7 mm to (138.1, 93.6)
