File: Motor Driver/reaction_wheel/power_supply.kicad_sch (KiCad schematic)
At the start: 22 parts, among them U2 TPS259531DSGR

Commit message: Schematic cleanup
Parts:
- added R10: 100k, Resistor_SMD:R_0603_1608Metric, symbol Device:R
- added R5: 0, Resistor_SMD:R_0603_1608Metric, symbol Device:R
- added TP1: AGND, TestPoint:TestPoint_Keystone_5000-5004_Miniature, symbol Connector:TestPoint
- added TP11: FLT_N, TestPoint:TestPoint_Keystone_5000-5004_Miniature, symbol Argus_RW_Library:5001
- added TP2: PGND, TestPoint:TestPoint_Keystone_5000-5004_Miniature, symbol Connector:TestPoint
- C8: value 3.3nF -> 22nF
- R7: value 100k -> 560k
- R8: value 1500 -> 1.5k
- TP3: value VBAT -> VIN
Connections:
- net PGND: now also R10.2, R5.2, TP2.1
- net at R7.2, U2.2 (EN_UVLO): now also R10.1
- net at U2.6 (FLT_N): now also TP11.1
- net VBAT renamed VIN
- new net AGND: R5.1, TP1.1
- no-connect marks 1 -> 0
Other:
- note added: "Grounding"
- note removed: "Reverse Polarity Protection"
- note removed: "can add a power switch to prevent in-rush current with soft start"
- note removed: "got rid of RPP"
- note removed: "used CAP ALUM POLY 330UF 20% 25V SMD"
- moved on the sheet: C15, C16, C17, C18, C19, C20, C21, C22, C7, C8, R7, R8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
