File: Motor Driver/reaction_wheel/reaction_wheel.kicad_pcb (KiCad board)
At the start: 4 copper layers, 34.5 x 40 mm, 44 parts, among them J1 Input Power, J4 Data Conn, J8 MOTOR_OUT, U1 MCF8315C1VQRGFRQ1, U2 TPS259531DSGR

Commit message: Schematic cleanup
Parts:
- added C23: 22uF, Capacitor_SMD:C_0603_1608Metric, F.Cu at (65.1, 110.5)
- added JP1: Jumper_2_Bridged, Jumper:SolderJumper-2_P1.3mm_Bridged_RoundedPad1.0x1.5mm, F.Cu at (103.9, 101.2)
- added JP2: Jumper_2_Bridged, Jumper:SolderJumper-2_P1.3mm_Bridged_RoundedPad1.0x1.5mm, F.Cu at (103.7, 105.0)
- added L1: 47uH, Inductor_SMD:L_0603_1608Metric, F.Cu at (68.2, 111.5)
- added R10: 100k, Resistor_SMD:R_0603_1608Metric, F.Cu at (59.6, 123.9)
- added TP1: AGND, TestPoint:TestPoint_Keystone_5000-5004_Miniature, F.Cu at (71.8, 95.0)
- added TP10: SPEED, TestPoint:TestPoint_Keystone_5000-5004_Miniature, F.Cu at (96.6, 106.1)
- added TP11: FLT_N, TestPoint:TestPoint_Keystone_5000-5004_Miniature, F.Cu at (100.7, 122.9)
- C8: value 3.3nF -> 22nF
- J1: value Input Power -> Molex Pico-Lock
- J4: value Data Conn -> 0522070860
- J8: value MOTOR_OUT -> Molex Pico-Lock
- R1, R9: value 5.1k -> 10k
- R7: value 100k -> 560k
- R8: value 1500 -> 1.5k
- TP3: value VBAT -> VIN
- moved C2 2.27 mm to (65.1, 109.0), turned to 180 degrees
- moved R7 1.76 mm to (60.2, 126.3)
- moved C1 1.22 mm to (70.3, 111.7), turned to -90 degrees
- moved TP3 0.89 mm to (56.0, 122.0)
Connections:
- C7 pad 1: VBAT -> VIN
- J1 pad 1: PGND -> VIN
- J1 pad 2: VBAT -> PGND
- J4 pad MP: AGND -> PGND
- R7 pad 1: VBAT -> VIN
- TP3 pad 1: VBAT -> VIN
- U1 pad 22: unconnected-(U1-NC-Pad22) -> AGND
- U1 pad 23: unconnected-(U1-NC-Pad23) -> AGND
- U1 pad 24: unconnected-(U1-NC-Pad24) -> AGND
- U1 pad 25: unconnected-(U1-NC-Pad25) -> AGND
- U1 pad 35: AGND -> /BRAKE
- U1 pad 5: /SW_BUCK -> Net-(U1-SW_BK)
- U2 pad 3: VBAT -> VIN
- U2 pad 4: VBAT -> VIN
- U2 pad 6: unconnected-(U2-FLT_N-Pad6) -> Net-(U2-FLT_N)
Routing:
- net /FB_BUCK: track 0.00 -> 4.49 mm
- net Net-(U1-SW_BK): track 0.00 -> 4.03 mm
- net AGND: track 18.0 -> 22.0 mm, vias 9 -> 6
- net VIN: track 0.00 -> 3.75 mm
- net VBAT: track 3.16 -> 0.00 mm
- net /CPL: track 2.70 -> 4.50 mm
- net Net-(U2-EN_UVLO): track 1.63 -> 3.20 mm
- net Net-(U1-DVDD): track 2.76 -> 2.06 mm
- net PGND: vias 28 -> 30
- added copper zone on F.Cu, net VIN
- removed copper zone on F.Cu, net VBAT
Other:
- board size 34.5 x 40 mm -> 34.6 x 38.1 mm
- copper layers 4 -> 2
- board text added: "Argus CubeSat Motor Driver V1.0"
- board text added: "CW"
- board text removed: "Filter"
- board text removed: "Grounding"
- board text removed: "chip"
