File: Motor Driver/reaction_wheel/reaction_wheel.kicad_sch (KiCad schematic)
At the start: 16 parts, among them U1 MCF8315C1VQRGFRQ1

Commit message: Schematic cleanup
Parts:
- added C23: 22uF, Capacitor_SMD:C_0603_1608Metric, symbol Device:C
- added JP1, JP2: Jumper_2_Bridged, Jumper:SolderJumper-2_P1.3mm_Bridged_RoundedPad1.0x1.5mm, symbol Jumper:Jumper_2_Bridged
- added L1: 47uH, Inductor_SMD:L_0603_1608Metric, symbol Device:L
- added TP10: SPEED, TestPoint:TestPoint_Keystone_5000-5004_Miniature, symbol Argus_RW_Library:5001
- R1, R9: value 5.1k -> 10k
Connections:
- net AGND: now also U1.22 (NC), U1.23 (NC), U1.24 (NC), U1.25 (NC), C23.2, JP1.1 (A), JP2.1 (A); no longer U1.35 (BRAKE)
- net DIR: now also JP2.2 (B)
- net FB_BUCK: now also C23.1, L1.2
- net SPEED: now also TP10.1
- net SW_BUCK: no longer names the net of U1.5 (SW_BK)
- net SW_BUCK: now also L1.1
- new net BRAKE: JP1.2 (B), U1.35 (BRAKE)
- no-connect marks 11 -> 5
Other:
- moved on the sheet: C1, C2, C3, C4, C5, C6, R1, R2, R3, R4, R6, R9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
