File: reaction_wheel/microcontroller_(1-axis_rw).kicad_sch (KiCad schematic)
At the start: 22 parts, among them J1 Conn_01x05_Pin, J2 Conn_01x04_Pin, J3 Conn_01x04_Pin, J4 Conn_01x04_Pin, J5 Conn_01x04_Pin, U6 STM32G474RETx

Commit message: things were not working on desktop
Parts:
- removed C2, C3, C4, C5, C6, C7, C8, C9: 100nF, symbol Device:C
- removed J1: Conn_01x05_Pin, symbol Connector:Conn_01x05_Pin
- removed J2, J3, J4, J5: Conn_01x04_Pin, symbol Connector:Conn_01x04_Pin
- removed R1, R2, R3, R4, R5, R6, R7, R8: 4.7k, symbol Device:R
- removed U6: STM32G474RETx, Package_QFP:LQFP-64_10x10mm_P0.5mm, symbol MCU_ST_STM32G4:STM32G474RETx
- added C10, C11, C12, C13, C14, C15, C16, C17: 100nF, symbol Device:C
- added J6: Conn_01x05_Pin, symbol Connector:Conn_01x05_Pin
- added J7: Conn_01x04_Pin, symbol Connector:Conn_01x04_Pin
- added J8: Conn_01x08_Pin, symbol Connector:Conn_01x08_Pin
- added J9: Conn_01x02_Pin, symbol Connector:Conn_01x02_Pin
- added R10, R11, R12, R13, R14, R15, R16, R9: 4.7k, symbol Device:R
- added U8: STM32G474RETx, Package_QFP:LQFP-64_10x10mm_P0.5mm, symbol MCU_ST_STM32G4:STM32G474RETx
Connections:
- net +12V: now also J9.2 (Pin_2)
- net +3V3: now also C11.1, C12.1, C13.1, C14.1, C15.1, C16.1, C17.1, J6.1 (Pin_1), J7.1 (Pin_1), R10.1, R11.1, R12.1, R13.1, R14.1, R15.1, R16.1, R9.1, U8.1 (VBAT), U8.16 (VDD), U8.28 (VREF+), U8.29 (VDDA), U8.32 (VDD), U8.48 (VDD), U8.64 (VDD)
- net GND: now also C10.2, C11.2, C12.2, C13.2, C14.2, C15.2, C16.2, C17.2, J6.3 (Pin_3), J7.2 (Pin_2), J8.2 (Pin_2), J8.4 (Pin_4), J8.6 (Pin_6), J8.8 (Pin_8), J9.1 (Pin_1), U8.15 (VSS), U8.27 (VSSA), U8.31 (VSS), U8.47 (VSS), U8.63 (VSS)
- net I2C1_SCL: now also J7.3 (Pin_3), J8.7 (Pin_7), R9.2, U8.59 (PB6)
- net I2C1_SDA: now also J7.4 (Pin_4), J8.5 (Pin_5), R10.2, U8.60 (PB7)
- net I2C2_SCL: now also R11.2
- net I2C2_SDA: now also R12.2
- net I2C3_SCL: now also R13.2
- net I2C3_SDA: now also R14.2
- net I2C4_SCL: now also R15.2
- net I2C4_SDA: now also R16.2
- net NRST: now also C10.1, J6.5 (Pin_5), U8.7 (PG10)
- net SWDCLK: now also J6.2 (Pin_2), U8.50 (PA14)
- net SWDIO: now also J6.4 (Pin_4), U8.49 (PA13)
- net nFAULT_1: now also J8.3 (Pin_3), U8.12 (PA0)
- new net ALARM: J8.1 (Pin_1)
Other:
- note added: "Motor Driver Connector (temp)"
- note added: "Power Supply??"
- note added: "molex pico clasp connector"
- note removed: "I2C all default config except I2C4; need to configure in SW so that SDA is PB9"

Commit message: Add files via upload
Parts:
- added C27: 10uF, symbol Device:C
- added C28: 10nF, symbol Device:C
- added C29, C30, C34: 22uF, symbol Device:C
- added C31: 4.7nF, symbol Device:C
- added C32: 0.1uF, symbol Device:C
- added C33: 2.2uF, symbol Device:C
- added C35: 1uF, symbol Device:C
- added J11: 5013310207, CONN_5013310000-SD_02_MOL, symbol molex_pico_clasp:5013310207
- added L3, L4: 1uH, symbol Device:L
- added R26: 26.1k, symbol Device:R
- added R29, R31: 100k, symbol Device:R
- added R30: 10k, symbol Device:R
- added R32: 18k, symbol Device:R
- added R33: 280k, symbol Device:R
- added R34: 20k, symbol Device:R
- added U10: TPS62902RPJR, QFN_902RPJR_TEX, symbol tps62902:TPS62902RPJR
- added U11: TPS61379QWRTERQ1, RTE0016K-IPC_A, symbol TPS62902RPJR_boost_converter:TPS61379QWRTERQ1
Connections:
- net +12V: now also C34.1, C35.1, R33.1, U11.10 (OUT), U11.9 (VO)
- net +3V3: now also C29.1, L3.2, U10.3 (VOS)
- net GND: now also C27.2, C28.2, C29.2, C30.2, C31.2, C33.2, C34.2, C35.2, J11.2, R26.2, R32.2, R34.2, U10.4 (GND), U11.17 (Thermal_Pad), U11.5 (MODE_SYNC), U11.7 (GND), U11.8 (GND)
- new net: C31.1, R30.2
- new net BST_Boost: C32.2, U11.2 (BST)
- new net COMP_Boost: R30.1, U11.14 (COMP)
- new net EN_Boost: R29.2, U11.15 (EN)
- new net FB_Boost: R33.2, R34.1, U11.13 (FB)
- new net FREQ_Boost: R32.1, U11.16 (FREQ)
- new net MODE_SCONF_Buck: R26.1, U10.7 (MODE/S-CONF)
- new net PG_Boost: R31.1, U11.11 (PG)
- new net SS_TR_Buck: C28.1, U10.8 (SS/TR)
- new net SW_Boost: C32.1, L4.2, U11.3 (SW), U11.4 (SW)
- new net SW_Buck: L3.1, U10.2 (SW)
- new net VBATT: C27.1, C30.1, J11.1, L4.1, R29.1, U10.5 (EN), U10.6 (VIN), U11.1 (VIN)
- new net VCC_Boost: C33.1, R31.2, U11.6 (VCC)
- no-connect marks 0 -> 3
Other:
- note added: "Battery Connector to ADCS Board"
- note added: "Boost Converter: Battery to +12V"
- note added: "Buck Converter: Battery to +3V3"
- note added: "For C27 (10uF cap), select a ceramic capacitor rated for at least 16V or 25V (X7R or X5R dielectric). Ceramic capacitors lose effective capacitance under DC bias voltage; a 10V-rated capacitor will drop below the minimum required capacitance when operating at 8V input."
- note added: "Power Supply to MD Board"
- note added: "SS/TR: do i need soft time start thing? for 1ms = 10nF else can leave open?"
- note removed: "Power Supply??"

Commit message: clean up sch, notes, added parts minus stlink
Parts:
- removed C27: 10uF, symbol Device:C
- removed C28: 10nF, symbol Device:C
- removed C29, C30, C34: 22uF, symbol Device:C
- removed C31: 4.7nF, symbol Device:C
- removed C32: 0.1uF, symbol Device:C
- removed C33: 2.2uF, symbol Device:C
- removed C35: 1uF, symbol Device:C
- removed J7: Conn_01x04_Pin, symbol Connector:Conn_01x04_Pin
- removed J8: Conn_01x08_Pin, symbol Connector:Conn_01x08_Pin
- removed J9: Conn_01x02_Pin, symbol Connector:Conn_01x02_Pin
- removed L3, L4: 1uH, symbol Device:L
- removed R26: 26.1k, symbol Device:R
- removed R29, R31: 100k, symbol Device:R
- removed R30: 10k, symbol Device:R
- removed R32: 18k, symbol Device:R
- removed R33: 280k, symbol Device:R
- removed R34: 20k, symbol Device:R
- removed U10: TPS62902RPJR, QFN_902RPJR_TEX, symbol tps62902:TPS62902RPJR
- removed U11: TPS61379QWRTERQ1, RTE0016K-IPC_A, symbol TPS62902RPJR_boost_converter:TPS61379QWRTERQ1
- added J10: SM04B-GHS-TB, CONN_SM04B-GHS-TB_JST, symbol SM04B_GHS_TB:SM04B-GHS-TB
- added J7: SM02B-GHS-TB, CONN_SM02B-GHS_JST, symbol SM02B_GHS_TB:SM02B-GHS-TB
- added J9: SM08B-GHS-TB, CONN_SM08B-GHS-TB_JST, symbol SM08B_GHS_TB:SM08B-GHS-TB
Connections:
- net +12V: now also J7.2
- net +3V3: now also J10.1
- net ALARM: now also J9.1
- net GND: now also J10.2, J7.1, J9.2, J9.4, J9.6, J9.8
- net I2C1_SCL: now also J10.3, J9.7
- net I2C1_SDA: now also J10.4, J9.5
- net nFAULT_1: now also J9.3
- no-connect marks 3 -> 0
Other:
- note added: "Battery to ADCS Board Connector"
- note added: "Found part, waiting to download part for free"
- note added: "Hall Sensor/Encoder Connectors"
- note added: "Microcontroller"
- note added: "Motor Driver Connector"
- note added: "Power Sources"
- note added: "Power Supply to Motor Driver Board"
- note removed: "Battery Connector to ADCS Board"
- note removed: "Boost Converter: Battery to +12V"
- note removed: "Buck Converter: Battery to +3V3"
- note removed: "For C27 (10uF cap), select a ceramic capacitor rated for at least 16V or 25V (X7R or X5R dielectric). Ceramic capacitors lose effective capacitance under DC bias voltage; a 10V-rated capacitor will drop below the minimum required capacitance when operating at 8V input."
- note removed: "Hall Sensor/Encoder Connectors (temp)"
- note removed: "Motor Driver Connector (temp)"
- note removed: "Power Supply to MD Board"
- note removed: "SS/TR: do i need soft time start thing? for 1ms = 10nF else can leave open?"
- moved on the sheet: C10, C11, C12, C13, C14, C15, C16, C17, J11, J6, R10, R11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

Commit message: added notes
Other:
- note added: "Note: Not sure how the board-to-board connector interacts with this board? I think the only thing I need is VBATT, should I change the Battery to ADCS board connector to the big board-to-board connector??"
Changed lines of the file:
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@@
+		)
+	)
+	(text "Note: Not sure how the board-to-board connector interacts with this board? \nI think the only thing I need is VBATT, should I change the Battery to ADCS board \nconnector to the big board-to-board connector??"
+		(exclude_from_sim no)
+		(at 181.102 47.498 0)
+		(effects
+			(font
+				(size 1.27 1.27)
+				(thickness 0.254)
+				(bold yes)
+			)
+			(justify left)
 		)
 	)

Commit message: need to fix erc errors
Parts:
- removed R11, R12, R13, R14, R15, R16: 4.7k, symbol Device:R
Connections:
- no-connect marks 0 -> 46
Other:
- moved on the sheet: R10, R9

Commit message: Add files via upload
Parts:
- added J1: QTH-030-01-L-D-A, symbol Connector_Generic:Conn_02x30_Odd_Even
Connections:
- net GND: now also J1.11 (Pin_11), J1.12 (Pin_12), J1.13 (Pin_13), J1.14 (Pin_14), J1.15 (Pin_15), J1.16 (Pin_16), J1.17 (Pin_17), J1.18 (Pin_18), J1.19 (Pin_19), J1.20 (Pin_20), J1.25 (Pin_25), J1.26 (Pin_26), J1.27 (Pin_27), J1.28 (Pin_28), J1.35 (Pin_35), J1.41 (Pin_41), J1.44 (Pin_44), J1.45 (Pin_45), J1.59 (Pin_59), J1.60 (Pin_60)
- net I2C1_SCL: now also J1.37 (Pin_37)
- net I2C1_SDA: now also J1.39 (Pin_39)
- net VBATT: now also J1.1 (Pin_1), J1.10 (Pin_10), J1.2 (Pin_2), J1.3 (Pin_3), J1.4 (Pin_4), J1.5 (Pin_5), J1.6 (Pin_6), J1.7 (Pin_7), J1.8 (Pin_8), J1.9 (Pin_9)
- new net +3V3_P: J1.21 (Pin_21), J1.22 (Pin_22), J1.23 (Pin_23), J1.24 (Pin_24)
- new net FREE_105: J1.55 (Pin_55)
- new net FREE_IO1: J1.47 (Pin_47)
- new net FREE_IO2: J1.49 (Pin_49)
- new net FREE_IO3: J1.51 (Pin_51)
- new net FREE_IO4: J1.53 (Pin_53)
- new net FREE_IO6: J1.57 (Pin_57)
- new net GPS_1PPS: J1.43 (Pin_43)
- new net SPIO_CLK: J1.29 (Pin_29)
- new net SPIO_MISO: J1.33 (Pin_33)
- new net SPIO_MOSI: J1.31 (Pin_31)
Other:
- note added: "need ALARM connection on stm32"

Commit message: got to layout
Parts:
- removed J10: SM04B-GHS-TB, CONN_SM04B-GHS-TB_JST, symbol SM04B_GHS_TB:SM04B-GHS-TB
- removed J11: 5013310207, CONN_5013310000-SD_02_MOL, symbol molex_pico_clasp:5013310207
- removed J6: Conn_01x05_Pin, symbol Connector:Conn_01x05_Pin
- removed J7: SM02B-GHS-TB, CONN_SM02B-GHS_JST, symbol SM02B_GHS_TB:SM02B-GHS-TB
- removed J9: SM08B-GHS-TB, CONN_SM08B-GHS-TB_JST, symbol SM08B_GHS_TB:SM08B-GHS-TB
- added J2: FTSH-105-01-L-DV, sidrishaLibrary:CON10_2X5_DU_FTSH_SAI, symbol FTSH-105-01-L-DV:FTSH-105-01-L-DV
- C10, C11, C12, C13, C14, C15, C16, C17: footprint (none) -> Capacitor_SMD:C_0603_1608Metric
- J1: footprint (none) -> sidrishaLibrary:SAMTEC-QTH-030-01-X-D-A
- R10, R9: footprint (none) -> Resistor_SMD:R_0603_1608Metric
Connections:
- net FREE_IO1 is gone; now on net RW_EN: J1.47 (Pin_47)
- net FREE_IO2 is gone; now on net RW_PWR_FLT: J1.49 (Pin_49)
- net FREE_IO4 is gone; now on net RW_MTR_ALRM: J1.53 (Pin_53)
- net nFAULT_1 is gone; now on net RW_MTR_FLT: U8.12 (PA0)
- net +3V3: now also J2.1
- net GND: now also J2.3, J2.5, J2.9
- net NRST: now also J2.10
- net SPIO_CLK: now also U8.19 (PA5)
- net SPIO_MISO: now also U8.20 (PA6)
- net SPIO_MOSI: now also U8.21 (PA7)
- net SWDCLK: now also J2.4
- net SWDIO: now also J2.2
- net VBATT: now also J1.01 (Pin_1), J1.02 (Pin_2), J1.03 (Pin_3), J1.04 (Pin_4), J1.05 (Pin_5), J1.06 (Pin_6), J1.07 (Pin_7), J1.08 (Pin_8), J1.09 (Pin_9); no longer J1.1 (Pin_1), J1.2 (Pin_2), J1.3 (Pin_3), J1.4 (Pin_4), J1.5 (Pin_5), J1.6 (Pin_6), J1.7 (Pin_7), J1.8 (Pin_8), J1.9 (Pin_9)
- net SPIO_NSS: now reaches J1.36 (Pin_36)
- net SPIO_NSS: now also U8.18 (PA4)
- net ADCS_EN: now reaches J1.38 (Pin_38)
- net ADCS_EN: now also U8.42 (PA8)
- net RW_PWR_FLT: now reaches U8.13 (PA1)
- net RW_MTR_ALRM: now reaches U8.14 (PA2)
- net RW_EN: now reaches U8.17 (PA3)
- net SWO: now reaches U8.56 (PB3)
- net SWO: now also J2.6
- net FREE_105 renamed RW_SCL
- net RW_SCL: now also R9.2, U8.59 (PB6)
- net FREE_IO3 renamed RW_MTR_FLT
- net FREE_IO6 renamed RW_SDA
- net RW_SDA: now also R10.2, U8.60 (PB7)
- net GPS_1PPS: no longer names the net of J1.43 (Pin_43)
- removed net I2C1_SCL: J1.37 (Pin_37), R9.2, U8.59 (PB6)
- removed net I2C1_SDA: J1.39 (Pin_39), R10.2, U8.60 (PB7)
- no-connect marks 46 -> 54
Other:
- added sheet Power (power.kicad_sch)
- note added: "ADCS_Chip_Select activeLow configure SPI in slave mode with hardware NSS"
- note added: "AltFn0"
- note added: "AltFn5 for SPI"
- note added: "BATT0_EN BATT1_EN BATT_ALRT"
- note added: "Board-to-board connector"
- note added: "GPS_1PPS"
- note added: "I2C1_SCL I2C1_SDA"
- note added: "NOTE: I2C all defualt config except I2C4; need to config in SW so SDA is PB9"
- note added: "Open: 40, 42, 46, 48, 50, 52"
- note added: "ST-Link Connector"
- note added: "eGPS_EN eGPS_TX eGPS_RX"
- note removed: "Battery to ADCS Board Connector"
- note removed: "Found part, waiting to download part for free"
- note removed: "Hall Sensor/Encoder Connectors"
- note removed: "Motor Driver Connector"
- note removed: "Note: Not sure how the board-to-board connector interacts with this board? I think the only thing I need is VBATT, should I change the Battery to ADCS board connector to the big board-to-board connector??"
- note removed: "Power Sources"
- note removed: "Power Supply to Motor Driver Board"
- note removed: "ST-Link Connector (temp)"
- note removed: "molex pico clasp connector"
- note removed: "need ALARM connection on stm32"
- moved on the sheet: C10, J1
