File: reaction_wheel/reaction_wheel.kicad_pcb (KiCad board)
At the start: 0 parts

Commit message: got to layout
Parts:
- added C1: 22uF, Capacitor_SMD:C_0603_1608Metric, F.Cu at (151.5, 110.5)
- added C10: 100nF, Capacitor_SMD:C_0603_1608Metric, F.Cu at (102.5, 85.5)
- added C11: 100nF, Capacitor_SMD:C_0603_1608Metric, F.Cu at (106.5, 69.0)
- added C12: 100nF, Capacitor_SMD:C_0603_1608Metric, F.Cu at (106.5, 71.5)
- added C13: 100nF, Capacitor_SMD:C_0603_1608Metric, F.Cu at (106.5, 74.0)
- added C14: 100nF, Capacitor_SMD:C_0603_1608Metric, F.Cu at (106.5, 76.5)
- added C15: 100nF, Capacitor_SMD:C_0603_1608Metric, F.Cu at (112.5, 68.5)
- added C16: 100nF, Capacitor_SMD:C_0603_1608Metric, F.Cu at (112.7, 71.5)
- added C17: 100nF, Capacitor_SMD:C_0603_1608Metric, F.Cu at (112.7, 74.0)
- added C2: 4.7nF, Capacitor_SMD:C_0603_1608Metric, F.Cu at (150.0, 121.0)
- added C3: 0.1uF, Capacitor_SMD:C_0603_1608Metric, F.Cu at (139.3, 124.0)
- added C4: 2.2uF, Capacitor_SMD:C_0603_1608Metric, F.Cu at (145.0, 133.0)
- added C5: 1uF, Capacitor_SMD:C_0603_1608Metric, F.Cu at (155.0, 129.0)
- added C6: 22uF, Capacitor_SMD:C_0603_1608Metric, F.Cu at (155.0, 132.5)
- added C7: 10uF, Capacitor_SMD:C_0603_1608Metric, F.Cu at (96.0, 129.2)
- added C8: 10nF, Capacitor_SMD:C_0603_1608Metric, F.Cu at (89.5, 134.2)
- added C9: 22uF, Capacitor_SMD:C_0603_1608Metric, F.Cu at (101.2, 132.2)
- added J1: QTH-030-01-L-D-A, sidrishaLibrary:SAMTEC-QTH-030-01-X-D-A, F.Cu at (160.5, 86.0)
- added J2: FTSH-105-01-L-DV, sidrishaLibrary:CON10_2X5_DU_FTSH_SAI, F.Cu at (160.5, 63.0)
- added L1: 1uH, Inductor_SMD:L_0603_1608Metric, F.Cu at (139.3, 121.0)
- added L2: 1uH, Inductor_SMD:L_0603_1608Metric, F.Cu at (99.7, 135.8)
- added R1: 100k, Resistor_SMD:R_0603_1608Metric, F.Cu at (144.0, 121.0)
- added R10: 4.7k, Resistor_SMD:R_0603_1608Metric, F.Cu at (126.2, 67.5)
- added R2: 10k, Resistor_SMD:R_0603_1608Metric, F.Cu at (150.0, 123.5)
- added R3: 100k, Resistor_SMD:R_0603_1608Metric, F.Cu at (149.0, 133.0)
- added R4: 18k, Resistor_SMD:R_0603_1608Metric, F.Cu at (144.0, 124.0)
- added R5: 280k, Resistor_SMD:R_0603_1608Metric, F.Cu at (155.0, 125.5)
- added R6: 20k, Resistor_SMD:R_0603_1608Metric, F.Cu at (159.5, 125.5)
- added R7: 26.1k, Resistor_SMD:R_0603_1608Metric, F.Cu at (89.5, 130.8)
- added R9: 4.7k, Resistor_SMD:R_0603_1608Metric, F.Cu at (126.2, 65.0)
- added U1: TPS61379QWRTERQ1, sidrishaLibrary:RTE0016K-IPC_B, F.Cu at (148.0, 128.5)
- added U2: TPS62902RPJR, sidrishaLibrary:QFN_902RPJR_TEX, F.Cu at (95.0, 132.0)
- added U8: STM32G474RETx, Package_QFP:LQFP-64_10x10mm_P0.5mm, F.Cu at (126.8, 86.8)
Routing:
- net /Power/PG_Boost: track 0.00 -> 8.45 mm
- net +3V3: track 0.00 -> 8.34 mm
- net /Power/SW_Buck: track 0.00 -> 6.16 mm
- net /Power/SS_TR_Buck: track 0.00 -> 4.83 mm
- net VBATT: track 0.00 -> 4.78 mm
- net /Power/EN_Boost: track 0.00 -> 4.62 mm
- net /Power/MODE_SCONF_Buck: track 0.00 -> 4.16 mm
- net /Power/COMP_Boost: track 0.00 -> 3.93 mm
- net /Power/FB_Boost: track 0.00 -> 2.85 mm
- net Net-(C2-Pad1): track 0.00 -> 2.52 mm
- net /Power/FREQ_Boost: track 0.00 -> 2.44 mm
- net /Power/VCC_Boost: track 0.00 -> 2.40 mm
- net /Power/SW_Boost: track 0.00 -> 0.50 mm
- net /Power/+12V: track 0.00 -> 0.50 mm
Other:
- board outline added: 90.2 x 95.9 mm
- copper layers 0 -> 2
